File: AS1802/TestBoard/TestBoard.kicad_pcb (KiCad board)
At the start: 4 copper layers, 99.6 x 60.7 mm, 45 parts, among them J1 Screw_Terminal_01x02, J2 PORTA, J3 JTAG, J4 Conn_01x06, J5 PORTB, J6 SPI, SW1 SW_Push, U1 74LVC573, U2 IS62LV256AL, U3 EPM240T100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

Commit message: VLIW ext4 progress
Parts:
- U2: footprint Package_SO:TSOP-I-28_11.8x8mm_P0.55mm -> TholinsStuff:TSOP-I-28_11.8x8mm_P0.55mm-weird-pin-order
Connections:
- U3 pad 26: N2 -> unconnected-(U3-IO1_26-Pad26)
- U3 pad 27: N1 -> unconnected-(U3-IO1_27-Pad27)
- U3 pad 28: N0 -> unconnected-(U3-IO1_28-Pad28)
- U3 pad 76: unconnected-(U3-IO2_76-Pad76) -> N0
- U3 pad 77: unconnected-(U3-IO2_77-Pad77) -> N1
- U3 pad 78: unconnected-(U3-IO2_78-Pad78) -> N2
Routing:
- net D1: track 97.0 -> 154.2 mm, vias 4 -> 6
- net D0: track 87.2 -> 139.3 mm
- net EXT: track 42.6 -> 87.1 mm, vias 2 -> 6
- net A6: track 39.0 -> 80.5 mm, vias 2 -> 4
- net A4: track 41.9 -> 77.9 mm, vias 2 -> 4
- net A5: track 41.7 -> 77.7 mm
- net A14: track 19.8 -> 55.1 mm, vias 0 -> 2
- net gpio: track 92.4 -> 126.5 mm, vias 3 -> 4
- net A13: track 23.9 -> 55.0 mm
- net A9: track 25.8 -> 56.4 mm
- net A12: track 28.2 -> 58.3 mm
- net A3: track 43.7 -> 73.5 mm, vias 2 -> 4
- net A8: track 30.1 -> 58.4 mm
- net SC1: track 42.5 -> 67.1 mm
- net A11: track 29.8 -> 53.6 mm
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Other:
- board text added: "AS1802 bring-up 0117"
- board text removed: "AS1802 bring-up 0109"
