File: MOS6502/TestBoard/TestBoard.kicad_sch (KiCad schematic)
At the start: 41 parts, among them J1 Screw_Terminal_01x02, J3 JTAG, J4 Conn_01x06, SW1 SW_Push, U2 IS62LV256AL, U3 EPM240T100, U4 W25Q32FVSS, U5 B2-CI2406, U6 MCP1319MT-29LE-OT, U7 AMS1117-1.8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

Commit message: Minor tweaks
Parts:
- added U1, U10, U11, U12, U13, U14, U15, U9: SK9822, TholinsStuff:SK9822-EC20, symbol TholinsStuff:SK9822
Connections:
- net +3V3: now also U1.4 (VCC), U10.4 (VCC), U11.4 (VCC), U12.4 (VCC), U13.4 (VCC), U14.4 (VCC), U15.4 (VCC), U9.4 (VCC)
- net GND: now also U1.3 (GND), U10.3 (GND), U11.3 (GND), U12.3 (GND), U13.3 (GND), U14.3 (GND), U15.3 (GND), U9.3 (GND)
- new net: U1.1 (SDI), U13.6 (SDO)
- new net: U1.2 (CKI), U13.5 (CKO)
- new net: U1.5 (CKO), U9.2 (CKI)
- new net: U1.6 (SDO), U9.1 (SDI)
- new net: U12.6 (SDO), U14.1 (SDI)
- new net: U12.5 (CKO), U14.2 (CKI)
- new net: U14.5 (CKO), U15.2 (CKI)
- new net: U14.6 (SDO), U15.1 (SDI)
- new net: U10.1 (SDI), U9.6 (SDO)
- new net: U10.2 (CKI), U9.5 (CKO)
- new net: U10.5 (CKO), U11.2 (CKI)
- new net: U10.6 (SDO), U11.1 (SDI)
- new net: U11.5 (CKO), U12.2 (CKI)
- new net: U11.6 (SDO), U12.1 (SDI)
- no-connect marks 22 -> 24
